File: pcb/barda.kicad_pcb (KiCad board)
At the start: 2 copper layers, 228.6 x 76.2 mm, 95 parts, among them J1 Conn_01x04, SW1 1U, SW10 1U, SW11 1U, SW12 1U, SW13 1.25U, SW14 1U, SW15 1U, SW16 1U, SW17 1U, SW18 1U, SW19 1U, SW2 1U, SW20 1U, SW21 1U, SW22 1U, SW23 1.75U, SW24 1U, SW25 1U, SW26 1U, SW27 1U, SW28 1U, SW29 1U, SW3 1U, SW30 1U, SW31 1U, SW32 1U, SW33 1.25U, SW34 1.25U, SW35 1U, SW36 1.25U, SW37 2.75U, SW38 1.25U, SW39 1U, SW4 1U, SW40 1.25U, SW41 1.75U, SW42 2.25U, SW5 1U, SW6 1U, SW7 1U, SW8 1U, SW9 1U, U1 HY0020

Commit message: Update Barda PCB and case design
Connections:
- net +3V3 renamed +3V0

Commit message: Update Barda case and PCB design
Parts:
- removed R2: 10k, Resistor_SMD:R_0402_1005Metric
- removed TS2: DFU, Button_Switch_SMD:SW_Push_SPST_NO_Alps_SKRK
- S1: value MSK12C02-HB -> MSK12C02-HB2.5
Connections:
- U1 pad K4: DFU -> unconnected-(U1-P0.20-PadK4)
Routing:
- net DFU: track 20.4 -> 0.00 mm, vias 2 -> 0
- net GND: track 6.57 -> 2.99 mm
- net +3V0: track 107.4 -> 104.5 mm
- net COL1: track 310.8 -> 309.6 mm
- net Net-(BT1--): vias 1838 -> 1841

Commit message: Update PCB and case for M2 4mm standoffs
Parts:
- removed BT1: CR1632, Smidr:BatteryHolder_Takachi_BS-S-1632
- added J2: Conn_01x02_Pin, Connector_PinHeader_2.54mm:PinHeader_1x02_P2.54mm_Vertical, B.Cu at (205.2, 119.1)
Connections:
- S1 pad 1: Net-(BT1--) -> unconnected-(S1-A-Pad1)
- S1 pad 2: GND -> Net-(J2-Pin_2)
- S1 pad 3: unconnected-(S1-C-Pad3) -> GND
Routing:
- net +3V0: track 104.5 -> 24.6 mm, vias 1 -> 0
- net Net-(J2-Pin_2): track 0.00 -> 18.6 mm
- net Net-(D42-A): track 7.79 -> 23.3 mm
- net Net-(D37-A): track 7.79 -> 23.3 mm
- net COL5: track 274.0 -> 266.5 mm
- net COL1: track 309.6 -> 302.9 mm
- net Net-(BT1--): track 2.84 -> 0.00 mm, vias 1841 -> 0
- net ROW6: track 234.1 -> 235.9 mm
- net GND: track 2.99 -> 4.68 mm
- removed copper zone on B.Cu, net Net-(BT1--)
- removed copper zone on F.Cu, net Net-(BT1--)
Other:
- outline, holes or cut-outs redrawn
