File: pcb/barda.kicad_pcb (KiCad board)
At the start: 2 copper layers, 228.6 x 76.2 mm, 93 parts, among them J1 Conn_01x04, J2 Conn_01x02_Pin, SW1 1U, SW10 1U, SW11 1U, SW12 1U, SW13 1.25U, SW14 1U, SW15 1U, SW16 1U, SW17 1U, SW18 1U, SW19 1U, SW2 1U, SW20 1U, SW21 1U, SW22 1U, SW23 1.75U, SW24 1U, SW25 1U, SW26 1U, SW27 1U, SW28 1U, SW29 1U, SW3 1U, SW30 1U, SW31 1U, SW32 1U, SW33 1.25U, SW34 1.25U, SW35 1U, SW36 1.25U, SW37 2.75U, SW38 1.25U, SW39 1U, SW4 1U, SW40 1.25U, SW41 1.75U, SW42 2.25U, SW5 1U, SW6 1U, SW7 1U, SW8 1U, SW9 1U, U1 HY0020

Commit message: Update Barda case and PCB designs
Other:
- outline, holes or cut-outs redrawn
- board text added: "Blad rev.0.1"
- board text removed: "Barda rev.0.1"
