File: pcb/barda.kicad_sch (KiCad schematic)
At the start: 93 parts, among them J1 Conn_01x04, SW1 1U, SW10 1U, SW11 1U, SW12 1U, SW13 1.25U, SW14 1U, SW15 1U, SW16 1U, SW17 1U, SW18 1U, SW19 1U, SW2 1U, SW20 1U, SW21 1U, SW22 1U, SW23 1.75U, SW24 1U, SW25 1U, SW26 1U, SW27 1U, SW28 1U, SW29 1U, SW3 1U, SW30 1U, SW31 1U, SW32 1U, SW33 1.25U, SW34 1.25U, SW35 1U, SW36 1.25U, SW37 2.75U, SW38 1.25U, SW39 1U, SW4 1U, SW40 1.25U, SW41 1.75U, SW42 2.25U, SW5 1U, SW6 1U, SW7 1U, SW8 1U, SW9 1U, U1 HY0020

Commit message: Update Barda PCB and case design
Connections:
- net +3V3 renamed +3V0
Changed lines of the file:
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@@
 	)
 	(junction
-		(at 185.42 153.67)
-		(diameter 0)
-		(color 0 0 0 0)
-	)
-	(junction
 		(at 218.44 50.8)
 		(diameter 0)
@@
 		(color 0 0 0 0)
 	)
+	(junction
+		(at 185.42 153.67)
+		(diameter 0)
+		(color 0 0 0 0)
+	)
 	(no_connect
 		(at 102.87 149.86)
@@
 	)
 	(symbol
-		(lib_id "power:+3V3")
+		(lib_id "power:+3V0")
 		(at 185.42 153.67 0)
 		(unit 1)
@@
 		(dnp no)
 		(fields_autoplaced yes)
-		(property "Reference" "#PWR09"
+		(property "Reference" "#PWR013"
 			(at 185.42 157.48 0)
 			(hide yes)
@@
 			)
 		)
-		(property "Value" "+3V3"
+		(property "Value" "+3V0"
 			(at 185.42 148.59 0)
 			(show_name no)
@@
 			)
 		)
-		(property "Description" "Power symbol creates a global label with name \"+3V3\""
+		(property "Description" "Power symbol creates a global label with name \"+3V0\""
 			(at 185.42 153.67 0)
 			(hide yes)
@@
 			(project "barda"
 				(path "/d92a227a-b637-3678-3dde-73c505c2d660"
-					(reference "#PWR09")
+					(reference "#PWR013")
 					(unit 1)
 				)
@@
 	)
 	(symbol
-		(lib_id "power:+3V3")
-		(at 120.65 142.24 0)
+		(lib_id "power:+3V0")
+		(at 96.52 170.18 0)
 		(unit 1)
 		(body_style 1)
@@
 		(dnp no)
 		(fields_autoplaced yes)
-		(property "Reference" "#PWR03"
-			(at 120.65 146.05 0)
+		(property "Reference" "#PWR010"
+			(at 96.52 173.99 0)
 			(hide yes)
 			(show_name no)
@@
 			)
 		)
-		(property "Value" "+3V3"
-			(at 120.65 137.16 0)
+		(property "Value" "+3V0"
+			(at 96.52 165.1 0)
 			(show_name no)
 			(do_not_autoplace no)
@@
 		)
 		(property "Footprint" ""
-			(at 120.65 142.24 0)
+			(at 96.52 170.18 0)
 			(hide yes)
 			(show_name no)
@@
 		)
 		(property "Datasheet" ""
-			(at 120.65 142.24 0)
+			(at 96.52 170.18 0)
 			(hide yes)
 			(show_name no)
@@
 			)
 		)
-		(property "Description" "Power symbol creates a global label with name \"+3V3\""
-			(at 120.65 142.24 0)
+		(property "Description" "Power symbol creates a global label with name \"+3V0\""
+			(at 96.52 170.18 0)
 			(hide yes)
 			(show_name no)
@@
 			(project "barda"
 				(path "/d92a227a-b637-3678-3dde-73c505c2d660"
-					(reference "#PWR03")
+					(reference "#PWR010")
 					(unit 1)
 				)
@@
 	)
 	(symbol
-		(lib_id "power:+3V3")
+		(lib_id "power:+3V0")
 		(at 107.95 137.16 0)
 		(unit 1)
@@
 		(dnp no)
 		(fields_autoplaced yes)
-		(property "Reference" "#PWR05"
+		(property "Reference" "#PWR011"
 			(at 107.95 140.97 0)
 			(hide yes)
@@
 			)
 		)
-		(property "Value" "+3V3"
+		(property "Value" "+3V0"
 			(at 107.95 132.08 0)
 			(show_name no)
@@
 			)
 		)
-		(property "Description" "Power symbol creates a global label with name \"+3V3\""
+		(property "Description" "Power symbol creates a global label with name \"+3V0\""
 			(at 107.95 137.16 0)
 			(hide yes)
@@
 			(project "barda"
 				(path "/d92a227a-b637-3678-3dde-73c505c2d660"
-					(reference "#PWR05")
+					(reference "#PWR011")
 					(unit 1)
 				)
@@
 	)
 	(symbol
+		(lib_id "power:+3V0")
+		(at 120.65 142.24 0)
+		(unit 1)
+		(body_style 1)
+		(exclude_from_sim no)
+		(in_bom yes)
+		(on_board yes)
+		(in_pos_files yes)
+		(dnp no)
+		(fields_autoplaced yes)
+		(property "Reference" "#PWR012"
+			(at 120.65 146.05 0)
+			(hide yes)
+			(show_name no)
+			(do_not_autoplace no)
+			(effects
+				(font
+					(size 1.27 1.27)
+				)
+			)
+		)
+		(property "Value" "+3V0"
+			(at 120.65 137.16 0)
+			(show_name no)
+			(do_not_autoplace no)
+			(effects
+				(font
+					(size 1.27 1.27)
+				)
+			)
+		)
+		(property "Footprint" ""
+			(at 120.65 142.24 0)
+			(hide yes)
+			(show_name no)
+			(do_not_autoplace no)
+			(effects
+				(font
+					(size 1.27 1.27)
+				)
+			)
+		)
+		(property "Datasheet" ""
+			(at 120.65 142.24 0)
+			(hide yes)
+			(show_name no)
+			(do_not_autoplace no)
+			(effects
+				(font
+					(size 1.27 1.27)
+				)
+			)
+		)
+		(property "Description" "Power symbol creates a global label with name \"+3V0\""
+			(at 120.65 142.24 0)
+			(hide yes)
+			(show_name no)
+			(do_not_autoplace no)
+			(effects
+				(font
+					(size 1.27 1.27)
+				)
+			)
+		)
+		(pin "1"
+		)
+		(instances
+			(project "barda"
+				(path "/d92a227a-b637-3678-3dde-73c505c2d660"
+					(reference "#PWR012")
+					(unit 1)
+				)
+			)
+		)
+	)
+	(symbol
 		(lib_id "Device:D")
 		(at 76.2 55.88 90)
@@
 					(unit 1)
 				)
-			)
-		)
-	)
-	(symbol
-		(lib_id "power:+3V3")
-		(at 96.52 170.18 0)
-		(unit 1)
-		(body_style 1)
-		(exclude_from_sim no)
-		(in_bom yes)
-		(on_board yes)
-		(in_pos_files yes)
-		(dnp no)
-		(fields_autoplaced yes)
-		(property "Reference" "#PWR07"
-			(at 96.52 173.99 0)
-			(hide yes)
-			(show_name no)
-			(do_not_autoplace no)
-			(effects
-				(font
-					(size 1.27 1.27)
-				)
-			)
-		)
-		(property "Value" "+3V3"
-			(at 96.52 165.1 0)
-			(show_name no)
-			(do_not_autoplace no)
-			(effects
-				(font
-					(size 1.27 1.27)
-				)
-			)
-		)
-		(property "Footprint" ""
-			(at 96.52 170.18 0)
-			(hide yes)
-			(show_name no)
-			(do_not_autoplace no)
-			(effects
-				(font
-					(size 1.27 1.27)
-				)
-			)
-		)
-		(property "Datasheet" ""
-			(at 96.52 170.18 0)
-			(hide yes)
-			(show_name no)
-			(do_not_autoplace no)
-			(effects
-				(font
-					(size 1.27 1.27)
-				)
-			)
-		)
-		(property "Description" "Power symbol creates a global label with name \"+3V3\""
-			(at 96.52 170.18 0)
-			(hide yes)
-			(show_name no)
-			(do_not_autoplace no)
-			(effects
-				(font
-					(size 1.27 1.27)
-				)
-			)
-		)
-		(pin "1"
-		)
-		(instances
-			(project "barda"
-				(path "/d92a227a-b637-3678-3dde-73c505c2d660"
-					(reference "#PWR07")
-					(unit 1)
-				)

Commit message: Update Barda case and PCB design
Parts:
- removed R2: 10k, Resistor_SMD:R_0402_1005Metric, symbol Device:R_Small
- removed TS2: DFU, Button_Switch_SMD:SW_Push_SPST_NO_Alps_SKRK, symbol Switch:SW_SPST
- S1: value MSK12C02-HB -> MSK12C02-HB2.5; JLCPCB Part # C431541 -> C47020937
Connections:
- net DFU: no longer names the net of U1.K4 (P0.20)
- no-connect marks 2 -> 3
Other:
- moved on the sheet: TS1

Commit message: Update PCB and case for M2 4mm standoffs
Parts:
- removed BT1: CR1632, Smidr:BatteryHolder_Takachi_BS-S-1632, symbol Device:Battery_Cell
- added J2: Conn_01x02_Pin, Connector_PinHeader_2.54mm:PinHeader_1x02_P2.54mm_Vertical, symbol Connector:Conn_01x02_Pin
Connections:
- net +3V0: now also J2.1 (Pin_1)
- net GND: now also S1.3 (C); no longer S1.2 (B)
- new net: J2.2 (Pin_2), S1.2 (B)
Changed lines of the file:
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@@
 	)
 	(no_connect
-		(at 102.87 149.86)
-	)
-	(no_connect
 		(at 162.56 137.16)
 	)
@@
 		(at 162.56 157.48)
 	)
+	(no_connect
+		(at 102.87 144.78)
+	)
 	(wire
 		(pts
@@
 	(wire
 		(pts
-			(xy 97.79 153.67) (xy 92.71 153.67)
-		)
-		(stroke
-			(width 0)
-			(type default)
-		)
-	)
-	(wire
-		(pts
 			(xy 215.9 76.2) (xy 220.98 76.2)
 		)
@@
 	(wire
 		(pts
+			(xy 102.87 149.86) (xy 102.87 153.67)
+		)
+		(stroke
+			(width 0)
+			(type default)
+		)
+	)
+	(wire
+		(pts
 			(xy 22.86 35.56) (xy 25.4 35.56)
 		)
@@
 	(wire
 		(pts
-			(xy 92.71 153.67) (xy 92.71 147.32)
-		)
-		(stroke
-			(width 0)
-			(type default)
-		)
-	)
-	(wire
-		(pts
 			(xy 91.44 50.8) (xy 91.44 63.5)
 		)
@@
 	(wire
 		(pts
+			(xy 87.63 144.78) (xy 85.09 144.78)
+		)
+		(stroke
+			(width 0)
+			(type default)
+		)
+	)
+	(wire
+		(pts
 			(xy 27.94 101.6) (xy 25.4 101.6)
 		)
@@
 	(wire
 		(pts
+			(xy 102.87 153.67) (xy 97.79 153.67)
+		)
+		(stroke
+			(width 0)
+			(type default)
+		)
+	)
+	(wire
+		(pts
 			(xy 177.8 50.8) (xy 177.8 52.07)
 		)
@@
 	(wire
 		(pts
+			(xy 85.09 147.32) (xy 92.71 147.32)
+		)
+		(stroke
+			(width 0)
+			(type default)
+		)
+	)
+	(wire
+		(pts
 			(xy 101.6 25.4) (xy 101.6 26.67)
 		)
@@
 	(wire
 		(pts
+			(xy 87.63 142.24) (xy 87.63 144.78)
+		)
+		(stroke
+			(width 0)
+			(type default)
+		)
+	)
+	(wire
+		(pts
 			(xy 152.4 50.8) (xy 152.4 52.07)
 		)
@@
 	(wire
 		(pts
-			(xy 102.87 144.78) (xy 107.95 144.78)
-		)
-		(stroke
-			(width 0)
-			(type default)
-		)
-	)
-	(wire
-		(pts
 			(xy 127 60.96) (xy 101.6 60.96)
 		)
@@
 	(symbol
 		(lib_id "power:+3V0")
-		(at 107.95 137.16 0)
+		(at 87.63 142.24 0)
 		(unit 1)
 		(body_style 1)
@@
 		(fields_autoplaced yes)
 		(property "Reference" "#PWR011"
-			(at 107.95 140.97 0)
+			(at 87.63 146.05 0)
 			(hide yes)
 			(show_name no)
@@
 		)
 		(property "Value" "+3V0"
-			(at 107.95 132.08 0)
+			(at 87.63 137.16 0)
 			(show_name no)
 			(do_not_autoplace no)
@@
 		)
 		(property "Footprint" ""
-			(at 107.95 137.16 0)
+			(at 87.63 142.24 0)
 			(hide yes)
 			(show_name no)
@@
 		)
 		(property "Datasheet" ""
-			(at 107.95 137.16 0)
+			(at 87.63 142.24 0)
 			(hide yes)
 			(show_name no)
@@
 		)
 		(property "Description" "Power symbol creates a global label with name \"+3V0\""
-			(at 107.95 137.16 0)
+			(at 87.63 142.24 0)
 			(hide yes)
 			(show_name no)
@@
 	)
 	(symbol
+		(lib_id "Connector:Conn_01x02_Pin")
+		(at 80.01 144.78 0)
+		(unit 1)
+		(body_style 1)
+		(exclude_from_sim no)
+		(in_bom yes)
+		(on_board yes)
+		(in_pos_files yes)
+		(dnp no)
+		(fields_autoplaced yes)
+		(property "Reference" "J2"
+			(at 80.645 139.7 0)
+			(show_name no)
+			(do_not_autoplace no)
+			(effects
+				(font
+					(size 1.27 1.27)
+				)
+			)
+		)
+		(property "Value" "Conn_01x02_Pin"
+			(at 80.645 142.24 0)
+			(show_name no)
+			(do_not_autoplace no)
+			(effects
+				(font
+					(size 1.27 1.27)
+				)
+			)
+		)
+		(property "Footprint" "Connector_PinHeader_2.54mm:PinHeader_1x02_P2.54mm_Vertical"
+			(at 80.01 144.78 0)
+			(hide yes)
+			(show_name no)
+			(do_not_autoplace no)
+			(effects
+				(font
+					(size 1.27 1.27)
+				)
+			)
+		)
+		(property "Datasheet" ""
+			(at 80.01 144.78 0)
+			(hide yes)
+			(show_name no)
+			(do_not_autoplace no)
+			(effects
+				(font
+					(size 1.27 1.27)
+				)
+			)
+		)
+		(property "Description" "Generic connector, single row, 01x02, script generated"
+			(at 80.01 144.78 0)
+			(hide yes)
+			(show_name no)
+			(do_not_autoplace no)
+			(effects
+				(font
+					(size 1.27 1.27)
+				)
+			)
+		)
+		(pin "1"
+		)
+		(pin "2"
+		)
+		(instances
+			(project "barda"
+				(path "/d92a227a-b637-3678-3dde-73c505c2d660"
+					(reference "J2")
+					(unit 1)
+				)
+			)
+		)
+	)
+	(symbol
 		(lib_name "GND_1")
 		(lib_id "power:GND")
@@
 					(unit 1)
 				)
-			)
-		)
-	)
-	(symbol
-		(lib_id "Device:Battery_Cell")
-		(at 107.95 142.24 0)
-		(unit 1)
-		(body_style 1)
-		(exclude_from_sim no)
-		(in_bom yes)
-		(on_board yes)
-		(in_pos_files yes)
-		(dnp no)
-		(fields_autoplaced yes)
-		(property "Reference" "BT1"
-			(at 111.76 139.1284 0)
-			(show_name no)
-			(do_not_autoplace no)
-			(effects
-				(font
-					(size 1.27 1.27)
-				)
-				(justify left)
-			)
-		)
-		(property "Value" "CR1632"
-			(at 111.76 141.6684 0)
-			(show_name no)
-			(do_not_autoplace no)
-			(effects
-				(font
-					(size 1.27 1.27)
-				)
-				(justify left)
-			)
-		)
-		(property "Footprint" "Smidr:BatteryHolder_Takachi_BS-S-1632"
-			(at 107.95 140.716 90)
-			(hide yes)
-			(show_name no)
-			(do_not_autoplace no)
-			(effects
-				(font
-					(size 1.27 1.27)
-				)
-			)
-		)
-		(property "Datasheet" ""
-			(at 107.95 140.716 90)
-			(hide yes)
-			(show_name no)
-			(do_not_autoplace no)
-			(effects
-				(font
-					(size 1.27 1.27)
-				)
-			)
-		)
-		(property "Description" "Single-cell battery"
-			(at 107.95 142.24 0)
-			(hide yes)
-			(show_name no)
-			(do_not_autoplace no)
-			(effects
-				(font
-					(size 1.27 1.27)
-				)
-			)
-		)
-		(property "Sim.Device" "V"
-			(at 107.95 142.24 0)
-			(hide yes)
-			(show_name no)
-			(do_not_autoplace no)
-			(effects
-				(font
-					(size 1.27 1.27)
-				)
-			)
-		)
-		(property "Sim.Type" "DC"
-			(at 107.95 142.24 0)
-			(hide yes)
-			(show_name no)
-			(do_not_autoplace no)
-			(effects
-				(font
-					(size 1.27 1.27)
-				)
-			)
-		)
-		(property "Sim.Pins" "1=+ 2=-"
-			(at 107.95 142.24 0)
-			(hide yes)
-			(show_name no)
-			(do_not_autoplace no)
-			(effects
-				(font
-					(size 1.27 1.27)
-				)
-			)
-		)
-		(property "LCSC Part" "C2902337"
-			(at 107.95 142.24 0)
-			(hide yes)
-			(show_name no)
-			(do_not_autoplace no)
-			(effects
-				(font
-					(size 1.27 1.27)
-				)
-			)
-		)
-		(pin "1"
-		)
-		(pin "2"
-		)
-		(instances
-			(project "barda"
-				(path "/d92a227a-b637-3678-3dde-73c505c2d660"
-					(reference "BT1")
-					(unit 1)
-				)
