File: pcb/barda_switch_plate.kicad_pcb (KiCad board)
At the start: 2 copper layers, 228.6 x 76.2 mm, 4 parts

Commit message: Update Barda case and PCB designs
Other:
- outline, holes or cut-outs redrawn
