File: pcb/blad_bottom_plate.kicad_pcb (KiCad board)
At the start: 2 copper layers, 228.6 x 76.2 mm, 7 parts

Commit message: Update PCB design
Parts:
- added G***: LOGO, Smidr:TechMark_FDK_HY0020, B.Cu at (127.8, 175.4)
Other:
- board text added: "Blað"
